Commit message: enable ros2 control and simulated camera

File: description/global_properties.xacro (robot description, xacro)
@@ -15,3 +15,7 @@
     <xacro:property name="caster_wheel_offset_x" value="-0.1146"/>
     <xacro:property name="caster_wheel_offset_z" value="${wheel_offset_z - wheel_diameter/2 + caster_wheel_diameter/2}"/>
+    <xacro:property name="camera_length" value="0.013"/>
+    <xacro:property name="camera_width" value="0.025"/>
+    <xacro:property name="camera_height" value="0.024"/>
+    <xacro:property name="camera_fov_deg" value="77"/>
 </robot>

File: description/lidar.xacro (robot description, xacro)
@@ -27,5 +27,5 @@
         <sensor name="laser" type="ray">
             <pose> 0 0 0 0 0 0</pose>
-            <visualize>true</visualize>
+            <visualize>false</visualize>
             <update_rate>10</update_rate>
             <ray>
@@ -47,5 +47,4 @@
                 <ros>
                     <argument>~/out:=scan</argument>
-                    <!-- <argument>-\-ros-args -\-remap ~/out:=scan</argument> -->
                 </ros>
                 <output_type>sensor_msgs/LaserScan</output_type>

File: description/robot.urdf.xacro (robot description, xacro)
@@ -1,6 +1,13 @@
 <?xml version="1.0"?>
 <robot xmlns:xacro="http://www.ros.org/wiki/xacro"  name="robot">
+    <xacro:arg name="use_ros2_control" default="true"/>
+    <xacro:if value="$(arg use_ros2_control)">
+        <xacro:include filename="ros2_control.xacro"/>
+    </xacro:if>
+    <xacro:unless value="$(arg use_ros2_control)">
+        <xacro:include filename="gazebo_control.xacro"/>
+    </xacro:unless>
     <xacro:include filename="robot_core.xacro"/>
-    <xacro:include filename="gazebo_control.xacro"/>
     <xacro:include filename="lidar.xacro"/>
+    <xacro:include filename="camera.xacro"/>
 </robot>

File: description/robot_core.xacro (robot description, xacro)
@@ -48,5 +48,5 @@
         <collision>
             <geometry>
-                <cylinder radius="${wheel_diameter/2}" length="${wheel_thickness}"/>
+                <sphere radius="${wheel_diameter/2}"/>
             </geometry>
         </collision>
@@ -74,5 +74,5 @@
         <collision>
             <geometry>
-                <cylinder radius="${wheel_diameter/2}" length="${wheel_thickness}"/>
+                <sphere radius="${wheel_diameter/2}"/>
             </geometry>
         </collision>
