Commit message: add base footprint link and enable lidar on sensors.launch

File: description/robot_core.xacro (robot description, xacro)
@@ -5,4 +5,11 @@
     <xacro:include filename="global_properties.xacro"/>
     <link name="base_link"/>
+    <joint name="base_footprint_joint" type="fixed">
+        <parent link="base_link"/>
+        <child link="base_footprint"/>
+        <origin xyz="0 0 0" rpy="0 0 0"/>
+    </joint>
+    <link name="base_footprint">
+    </link>
     <!-- Main Stack Link -->
     <joint name="main_stack_joint" type="fixed">
