Commit message: first simulation configurations

File: description/robot.urdf.xacro (robot description, xacro)
@@ -2,3 +2,4 @@
 <robot xmlns:xacro="http://www.ros.org/wiki/xacro"  name="robot">
     <xacro:include filename="robot_core.xacro"/>
+    <xacro:include filename="gazebo_control.xacro"/>
 </robot>

File: description/robot_core.xacro (robot description, xacro)
@@ -3,34 +3,38 @@
     <xacro:include filename="materials.xacro"/>
     <xacro:include filename="inertial_macros.xacro"/>
-    <link name="base_link">
-    </link>
+    <xacro:include filename="global_properties.xacro"/>
+    <link name="base_link"/>
+    <!-- Main Stack Link -->
     <joint name="main_stack_joint" type="fixed">
         <parent link="base_link"/>
         <child link="main_stack"/>
-        <origin xyz="-0.180 0 0"/>
+        <origin xyz="0 0 0"/>
     </joint>
     <link name="main_stack">
         <visual>
-            <origin xyz="0.125 0 0.09"/>
+            <origin xyz="-0.05 0 ${chassis_height/2}"/>
             <geometry>
-                <box size="0.25 0.25 0.18"/>
+                <box size="${chassis_length} ${chassis_width} ${chassis_height}"/>
             </geometry>
             <material name="white"/>
         </visual>
         <collision>
-            <origin xyz="0.125 0 0.09"/>
+            <origin xyz="-0.05 0 ${chassis_height/2}"/>
             <geometry>
-                <box size="0.25 0.25 0.18"/>
+                <box size="${chassis_length} ${chassis_width} ${chassis_height}"/>
             </geometry>
         </collision>
-        <xacro:inertial_box mass="0.5" x="0.25" y="0.25" z="0.18">
-            <origin xyz="0.125 0 0.09" rpy="0 0 0"/>
+        <xacro:inertial_box mass="0.5" x="${chassis_length}" y="${chassis_width}" z="${chassis_height}">
+            <origin xyz="-0.05 0 ${chassis_height/2}" rpy="0 0 0"/>
         </xacro:inertial_box>
     </link>
+    <gazebo reference="main_stack">
+        <material>Gazebo/White</material>
+    </gazebo>
     <!-- LEFT WHEEL LINK -->
     <joint name="left_wheel_joint" type="continuous">
         <parent link="base_link"/>
         <child link="left_wheel"/>
-        <origin xyz="0 0.145 0" rpy="-${pi/2} 0 0"/>
+        <origin xyz="${wheel_offset_x} ${wheel_offset_y} ${wheel_offset_z}" rpy="-${pi/2} 0 0"/>
         <axis xyz="0 0 1"/>
     </joint>
@@ -38,5 +42,5 @@
         <visual>
             <geometry>
-                <cylinder radius="0.05" length="0.02"/>
+                <cylinder radius="${wheel_diameter/2}" length="${wheel_thickness}"/>
             </geometry>
             <material name="blue"/>
@@ -44,22 +48,25 @@
         <collision>
             <geometry>
-                <cylinder radius="0.05" length="0.02"/>
+                <cylinder radius="${wheel_diameter/2}" length="${wheel_thickness}"/>
             </geometry>
         </collision>
-        <xacro:inertial_cylinder mass="0.1" length="0.02" radius="0.05">
+        <xacro:inertial_cylinder mass="${wheel_mass}" radius="${wheel_diameter/2}" length="${wheel_thickness}">
             <origin xyz="0 0 0" rpy="0 0 0"/>
         </xacro:inertial_cylinder>
     </link>
+    <gazebo reference="left_wheel">
+        <material>Gazebo/Blue</material>
+    </gazebo>
     <!-- RIGHT WHEEL LINK -->
     <joint name="right_wheel_joint" type="continuous">
         <parent link="base_link"/>
         <child link="right_wheel"/>
-        <origin xyz="0 -0.145 0" rpy="${pi/2} 0 0"/>
-        <axis xyz="0 0 1"/>
+        <origin xyz="${wheel_offset_x} ${-wheel_offset_y} ${wheel_offset_z}" rpy="${pi/2} 0 0"/>
+        <axis xyz="0 0 -1"/>
     </joint>
     <link name="right_wheel">
         <visual>
             <geometry>
-                <cylinder radius="0.05" length="0.02"/>
+                <cylinder radius="${wheel_diameter/2}" length="${wheel_thickness}"/>
             </geometry>
             <material name="blue"/>
@@ -67,21 +74,24 @@
         <collision>
             <geometry>
-                <cylinder radius="0.05" length="0.02"/>
+                <cylinder radius="${wheel_diameter/2}" length="${wheel_thickness}"/>
             </geometry>
         </collision>
-        <xacro:inertial_cylinder mass="0.1" length="0.02" radius="0.05">
+        <xacro:inertial_cylinder mass="${wheel_mass}" radius="${wheel_diameter/2}" length="${wheel_thickness}">
             <origin xyz="0 0 0" rpy="0 0 0"/>
         </xacro:inertial_cylinder>
     </link>
+    <gazebo reference="right_wheel">
+        <material>Gazebo/Blue</material>
+    </gazebo>
     <!-- CASTER WHEEL LINK -->
     <joint name="caster_wheel_link" type="fixed">
         <parent link="main_stack"/>
         <child link="caster_wheel"/>
-        <origin xyz="0.05 0 0"/>
+        <origin xyz="${caster_wheel_offset_x} 0 ${caster_wheel_offset_z}"/>
     </joint>
     <link name="caster_wheel">
         <visual>
             <geometry>
-                <sphere radius="0.05"/>
+                <sphere radius="${caster_wheel_diameter/2}"/>
             </geometry>
             <material name="black"/>
@@ -89,10 +99,15 @@
         <collision>
             <geometry>
-                <sphere radius="0.05"/>
+                <sphere radius="${caster_wheel_diameter/2}"/>
             </geometry>
         </collision>
-        <xacro:inertial_sphere mass="0.1" radius="0.05">
+        <xacro:inertial_sphere mass="${caster_wheel_mass}" radius="${caster_wheel_diameter/2}">
             <origin xyz="0 0 0" rpy="0 0 0"/>
         </xacro:inertial_sphere>
     </link>
+    <gazebo reference="caster_wheel">
+        <material>Gazebo/Black</material>
+        <mu1 value="0.0001"/>
+        <mu2 value="0.0001"/>
+    </gazebo>
 </robot>

Commit message: reorganize project

File: description/robot.urdf.xacro (robot description, xacro)
@@ -1,4 +1,5 @@
 <?xml version="1.0"?>
 <robot xmlns:xacro="http://www.ros.org/wiki/xacro"  name="robot">
+    <xacro:arg name="sim_mode" default="false"/>
     <xacro:arg name="use_ros2_control" default="true"/>
     <xacro:if value="$(arg use_ros2_control)">

File: description/robot_core.xacro (robot description, xacro)
@@ -5,4 +5,11 @@
     <xacro:include filename="global_properties.xacro"/>
     <link name="base_link"/>
+    <joint name="base_footprint_joint" type="fixed">
+        <parent link="base_link"/>
+        <child link="base_footprint"/>
+        <origin xyz="0 0 0" rpy="0 0 0"/>
+    </joint>
+    <link name="base_footprint">
+    </link>
     <!-- Main Stack Link -->
     <joint name="main_stack_joint" type="fixed">

File: description/ros2_control.xacro (robot description, xacro)
@@ -2,35 +2,61 @@
 <robot xmlns:xacro="http://www.ros.org/wiki/xacro">
     <xacro:include filename="global_properties.xacro"/>
-    <ros2_control name="RealRobot" type="system">
-        <hardware>
-            <plugin>diffdrive_arduino/DiffDriveArduinoHardware</plugin>
-            <param name="left_wheel_name">left_wheel_joint</param>
-            <param name="right_wheel_name">right_wheel_joint</param>
-            <param name="loop_rate">1.0</param>
-            <param name="device">/dev/ttyUSB0</param>
-            <param name="baud_rate">115200</param>
-            <param name="timeout_ms">1000</param>
-            <param name="enc_counts_per_rev">898</param>
-        </hardware>
-        <joint name="left_wheel_joint">
-            <command_interface name="velocity">
-                <param name="min">-10</param>
-                <param name="max">10</param>
-            </command_interface>
-            <state_interface name="position"/>
-            <state_interface name="velocity"/>
-        </joint>
-        <joint name="right_wheel_joint">
-            <command_interface name="velocity">
-                <param name="min">-10</param>
-                <param name="max">10</param>
-            </command_interface>
-            <state_interface name="position"/>
-            <state_interface name="velocity"/>
-        </joint>
-    </ros2_control>
+    <xacro:unless value="$(arg sim_mode)">
+        <ros2_control name="RealRobot" type="system">
+            <hardware>
+                <plugin>diffdrive_arduino/DiffDriveArduinoHardware</plugin>
+                <param name="left_wheel_name">left_wheel_joint</param>
+                <param name="right_wheel_name">right_wheel_joint</param>
+                <param name="loop_rate">1.0</param>
+                <param name="device">/dev/ttyUSB0</param>
+                <param name="baud_rate">115200</param>
+                <param name="timeout_ms">1000</param>
+                <param name="enc_counts_per_rev">898</param>
+            </hardware>
+            <joint name="left_wheel_joint">
+                <command_interface name="velocity">
+                    <param name="min">-10</param>
+                    <param name="max">10</param>
+                </command_interface>
+                <state_interface name="position"/>
+                <state_interface name="velocity"/>
+            </joint>
+            <joint name="right_wheel_joint">
+                <command_interface name="velocity">
+                    <param name="min">-10</param>
+                    <param name="max">10</param>
+                </command_interface>
+                <state_interface name="position"/>
+                <state_interface name="velocity"/>
+            </joint>
+        </ros2_control>
+    </xacro:unless>
+    <xacro:if value="$(arg sim_mode)">
+        <ros2_control name="GazeboSystem" type="system">
+            <hardware>
+                <plugin>gazebo_ros2_control/GazeboSystem</plugin>
+            </hardware>
+            <joint name="left_wheel_joint">
+                <command_interface name="velocity">
+                    <param name="min">-10</param>
+                    <param name="max">10</param>
+                </command_interface>
+                <state_interface name="velocity"/>
+                <state_interface name="position"/>
+            </joint>
+            <joint name="right_wheel_joint">
+                <command_interface name="velocity">
+                    <param name="min">-10</param>
+                    <param name="max">10</param>
+                </command_interface>
+                <state_interface name="velocity"/>
+                <state_interface name="position"/>
+            </joint>
+        </ros2_control>
+    </xacro:if>
     <gazebo>
         <plugin name="gazebo_ros2_control" filename="libgazebo_ros2_control.so">
             <parameters>$(find penelobot)/config/my_controllers.yaml</parameters>
+            <parameters>$(find penelobot)/config/gaz_ros2_ctl_use_sim.yaml</parameters>
         </plugin>
     </gazebo>
