Commit message: cleanup and tof camera added

File: description/camera.xacro (robot description, xacro)
@@ -5,5 +5,5 @@
         <parent link="base_link"/>
         <child link="camera_link"/>
-        <origin xyz="${0.029+camera_length} 0 ${0.15015-camera_height/2}" rpy="0 0 0"/>
+        <origin xyz="${0.029+camera_length} 0 ${0.15015-camera_height/2}" rpy="${pi} 0 0"/>
     </joint>
     <link name="camera_link">

File: description/global_properties.xacro (robot description, xacro)
@@ -5,9 +5,9 @@
     <xacro:property name="chassis_height" value="0.155"/>
     <xacro:property name="chassis_mass" value="1.5"/>
-    <xacro:property name='wheel_diameter' value='0.068'/>
+    <xacro:property name='wheel_diameter' value='0.0675'/>
     <xacro:property name="wheel_thickness" value="0.027"/>
     <xacro:property name="wheel_mass" value="0.05"/>
     <xacro:property name="wheel_offset_x" value="0.0"/>
-    <xacro:property name="wheel_offset_y" value="0.105"/>
+    <xacro:property name="wheel_offset_y" value="0.105"/> <!-- Offset is slightly lower than the wheel center to account for wheel pointof contact -->
     <xacro:property name="wheel_offset_z" value="-0.031"/>
     <xacro:property name="caster_wheel_diameter" value="0.038"/>
@@ -19,3 +19,9 @@
     <xacro:property name="camera_height" value="0.024"/>
     <xacro:property name="camera_fov_deg" value="77"/>
+    <xacro:property name="tof_camera_length" value="0.020" />
+    <xacro:property name="tof_camera_width" value="0.040" />
+    <xacro:property name="tof_camera_height" value="0.020" />
+    <!-- The horizontal FOV for the 100x100 mode is typically around 80-90 degrees.
+         We can calculate it from the intrinsics if needed, but 85 is a good start. -->
+    <xacro:property name="tof_camera_fov_deg" value="85.0" />
 </robot>

File: description/robot.urdf.xacro (robot description, xacro)
@@ -12,3 +12,4 @@
     <xacro:include filename="lidar.xacro"/>
     <xacro:include filename="camera.xacro"/>
+    <xacro:include filename="tof_camera.xacro"/>
 </robot>

File: description/ros2_control.xacro (robot description, xacro)
@@ -9,6 +9,6 @@
                 <param name="right_wheel_name">right_wheel_joint</param>
                 <param name="loop_rate">1.0</param>
-                <param name="device">/dev/ttyACM0</param>
-                <param name="baud_rate">115200</param>
+                <param name="device">/dev/serial/by-id/usb-Espressif_USB_JTAG_serial_debug_unit_64:E8:33:83:BA:2C-if00</param>
+                <param name="baud_rate">230400</param>
                 <param name="timeout_ms">1000</param>
                 <param name="enc_counts_per_rev">1975</param>
