Commit message: update lidar confs

File: description/lidar.xacro (robot description, xacro)
@@ -5,5 +5,5 @@
         <parent link="main_stack"/>
         <child link="laser_frame"/>
-        <origin xyz="-0.02 0 ${chassis_height+0.046}" rpy="0 0 0"/>
+        <origin xyz="-0.02 0 ${chassis_height+0.046}" rpy="${pi} 0 0"/>
     </joint>
     <link name="laser_frame">
